File: umidade.kicad_pcb (KiCad board)
At the start: 2 copper layers, 97.3 x 48.8 mm, 38 parts, among them IC1 ATMEGA328-P, J1 JACK_2P, J2 SENSOR1, J3 SENSOR2, J4 TEMP, J5 AVCC/AREF, SW1 SW_PUSH, SW2 SW_PUSH, U1 AMS1117, U2 ESP-12E, U3 AMS1117, X1 16MHz

Commit message: 2 commit
Parts:
- added C7: 100nF, Capacitors_SMD:C_1206_HandSoldering, F.Cu at (77.1, 111.1)
- added P1: CONN_01X06, Pin_Headers:Pin_Header_Straight_1x06, F.Cu at (135.2, 111.3)
- added SW3: SPDT, Buttons_Switches_THT:SW_Micro_SPST, F.Cu at (97.2, 85.8)
- C1, C2, C5, C6: value 10μF -> 22μF
- R1, R3, R4, R5: value 560R -> 10K
Connections:
- IC1 pad 2: RXD-ATMEGA -> ESP_GPIO16
- IC1 pad 3: TXD-ATMEGA -> (no net)
- R1 pad 2: 3.3V -> Net-(C7-Pad1)
- R3 pad 2: 3.3V -> Net-(C7-Pad1)
- R5 pad 1: 3.3V -> Net-(C7-Pad1)
- SW1 pad 2: 3.3V -> Net-(C7-Pad1)
- U2 pad 15: TXD-ATMEGA -> ESP_RXD
- U2 pad 16: RXD-ATMEGA -> ESP_TXD
- U2 pad 4: (no net) -> ESP_GPIO16
- U2 pad 8: 3.3V -> Net-(C7-Pad1)
Routing:
- net Net-(C7-Pad1): track 0.00 -> 67.2 mm
- net ESP_TXD: track 0.00 -> 62.1 mm
- net ESP_RXD: track 0.00 -> 55.3 mm
- net VCC_FTDI: track 0.00 -> 51.8 mm
- net ESP_GPIO16: track 0.00 -> 31.6 mm, vias 0 -> 1
- net TXD-ATMEGA: track 23.5 -> 0.00 mm
- net RXD-ATMEGA: track 22.7 -> 0.00 mm
- net 3.3V: track 71.2 -> 50.3 mm, vias 0 -> 1
- net GND: track 73.7 -> 72.0 mm, vias 16 -> 18
Other:
- board size 97.3 x 48.8 mm -> 99.2 x 51.1 mm
- board text added: "FPGA/FTDI"
- board text added: "GND"
- board text added: "PROG"
- board text added: "RX"
- board text added: "TX"
- board text added: "VCC"

Commit message: revisao mais profissional
Signed-off-by: Gabriel <gabrielnl@gmail.com>
Parts:
- RV1: value 90K -> 100K
Connections:
- net 5V renamed +5V
- net GND renamed Earth
- net V0 renamed Net-(DS1-Pad3)
- net VCC_FTDI renamed VCC
- C1 pad 1: 3.3V -> +3V3
- D1 pad 2: 3.3V -> Net-(C7-Pad1)
- SW3 pad 1: 3.3V -> +3V3
- U1 pad 2: 3.3V -> +3V3
Routing:
- net 3.3V: track 50.3 -> 0.00 mm, vias 1 -> 0
- net +3V3: track 0.00 -> 33.1 mm, vias 0 -> 2
- net Net-(C7-Pad1): track 67.2 -> 86.9 mm, vias 0 -> 2
- net Earth: track 72.0 -> 84.0 mm
