File: umidade.sch (KiCad schematic (older format))
At the start: 41 parts, among them IC1 ATMEGA328-P, J1 JACK_2P, J2 SENSOR1, J3 SENSOR2, J4 TEMP, J5 AVCC/AREF, P1 CONN_01X06, SW1 SW_PUSH, SW2 SW_PUSH, SW3 SPDT, U1 AMS1117, U2 ESP-12E, U3 AMS1117, X1 16MHz

Commit message: 2nd commit?
Signed-off-by: Gabriel <gabrielnl@gmail.com>
Other:
- note added: "ATMEGA"
- note added: "Header para o FTDI"
- note added: "LCD"
- note added: "Módulo ESP"
- note added: "Potência e Reguladores de Tensão"
- note added: "Sensor de Temperatura"
- note added: "Sensores de umidade"
- moved on the sheet: J4, R9
Changed lines of the file:
@@
 L HEADER_3 J4
 U 1 1 5981200B
-P 10400 6450
-F 0 "J4" H 10400 6650 60  0000 C CNN
-F 1 "TEMP" H 10400 6250 60  0000 C CNN
-F 2 "Terminal_Blocks:TerminalBlock_Pheonix_MPT-2.54mm_3pol" H 10400 6450 60  0001 C CNN
-F 3 "" H 10400 6450 60  0000 C CNN
-	1    10400 6450
-	1    0    0    -1
-$EndComp
-Wire Wire Line
-	9500 6550 10300 6550
+P 12700 8400
+F 0 "J4" H 12700 8600 60  0000 C CNN
+F 1 "TEMP" H 12700 8200 60  0000 C CNN
+F 2 "Terminal_Blocks:TerminalBlock_Pheonix_MPT-2.54mm_3pol" H 12700 8400 60  0001 C CNN
+F 3 "" H 12700 8400 60  0000 C CNN
+	1    12700 8400
+	1    0    0    -1
+$EndComp
+Wire Wire Line
+	11800 8500 12600 8500
 $Comp
 L R R9
 U 1 1 59812691
-P 9700 6450
-F 0 "R9" V 9780 6450 50  0000 C CNN
-F 1 "4.7K" V 9700 6450 50  0000 C CNN
-F 2 "Resistors_SMD:R_0805_HandSoldering" V 9630 6450 50  0001 C CNN
-F 3 "" H 9700 6450 50  0000 C CNN
-	1    9700 6450
+P 12000 8400
+F 0 "R9" V 12080 8400 50  0000 C CNN
+F 1 "4.7K" V 12000 8400 50  0000 C CNN
+F 2 "Resistors_SMD:R_0805_HandSoldering" V 11930 8400 50  0001 C CNN
+F 3 "" H 12000 8400 50  0000 C CNN
+	1    12000 8400
 	0    1    1    0
 $EndComp
@@
 Text GLabel 12700 4000 2    60   Input ~ 0
 GND
-Text GLabel 10300 6350 0    60   Input ~ 0
+Text GLabel 12600 8300 0    60   Input ~ 0
 GND
 Text GLabel 12050 4800 2    60   Input ~ 0
@@
 PD2
 Wire Wire Line
-	10300 6450 9850 6450
-Wire Wire Line
-	9500 6550 9500 6450
-Wire Wire Line
-	9500 6450 9550 6450
-Text GLabel 9500 6550 0    60   Input ~ 0
+	12600 8400 12150 8400
+Wire Wire Line
+	11800 8500 11800 8400
+Wire Wire Line
+	11800 8400 11850 8400
+Text GLabel 11800 8500 0    60   Input ~ 0
 5V
 Text GLabel 8600 2400 2    60   Input ~ 0
@@
 ADC4
 NoConn ~ 10950 4700
-Text GLabel 9900 6150 1    60   Input ~ 0
+Text GLabel 12200 8100 1    60   Input ~ 0
 PB2
 Wire Wire Line
-	9900 6150 9900 6450
-Connection ~ 9900 6450
+	12200 8100 12200 8400
+Connection ~ 12200 8400
 NoConn ~ 10950 3850
 $Comp
@@
 $EndComp
 Connection ~ 6300 7450
+Text Notes 12750 5500 0    60   ~ 0
+Sensores de umidade
+Text Notes 11500 3500 0    60   ~ 0
+ATMEGA
+Text Notes 10950 1500 0    60   ~ 0
+LCD
+Text Notes 4550 2700 0    60   ~ 0
+Potência e Reguladores de Tensão
+Text Notes 3250 5550 0    60   ~ 0
+Header para o FTDI
+Text Notes 12550 8000 0    60   ~ 0
+Sensor de Temperatura
+Text Notes 7000 8400 0    60   ~ 0
+Módulo ESP
 $EndSCHEMATC

Commit message: revisao mais profissional
Signed-off-by: Gabriel <gabrielnl@gmail.com>
Parts:
- RV1: value 90K -> 100K
Connections:
- net at C7.1, R1.2, R3.2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: now also D1.2 (A)
- net 3.3V renamed +3V3
- net +3V3: no longer D1.2 (A)
- net 5V renamed +5V
- net GND renamed Earth
- net V0: no longer names the net of DS1.3 (VO), RV1.2
- net VCC_FTDI renamed VCC
Other:
- note added: "Circuito alimentado através de um jack 2p\nRegulador de 5v para os sensores e ATMEGA\nRegulador de 3.3v para o ESP8266"
- note added: "O clock será gerado através de um oscilador\nO circuito dispõe de um header para determinar AVCC e AREF\nReset através de pushbutton"
- note added: "O dispositivo real será conectado no circuito através de um Header 16x1\nO potenciômetro regula o backlight"
- note added: "Os sensores serão conectados no circuito através dos headers"
- note added: "Programação do ESP8266 via FTDI\nChaveamento para alimentação do Regulador de Tensão do Circuito ou do FTDI\nLED para indicar que o circuito do ESP está funcionando\nO GPIO16 está conectado na ATMEGA"
- moved on the sheet: C1, C2, C3, C4, C5, C6, C7, D1, D2, D3, D4, D5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
